Commit message: fixed capitolization and inertial issues

File: Robot/Robot.URDF (robot description, URDF)
Before this commit: robot Robot, 5 links, 4 joints
Links:
- link Chassis: geometry collision mesh filename=package://Robot/collisionSTL/Chassis.STL; visual mesh filename=package://Robot/visualSTL/Chassis.STL
- link FL Wheel: geometry collision mesh filename=package://Robot/collisionSTL/FL Wheel.STL; visual mesh filename=package://Robot/visualSTL/FL Wheel.STL
- link FR Wheel: geometry collision mesh filename=package://Robot/collisionSTL/FR Wheel.STL; visual mesh filename=package://Robot/visualSTL/FR Wheel.STL
- link RL Wheel: geometry collision mesh filename=package://Robot/collisionSTL/RL Wheel.STL; visual mesh filename=package://Robot/visualSTL/RL Wheel.STL
- link RR Wheel: geometry collision mesh filename=package://Robot/collisionSTL/RR Wheel.STL; visual mesh filename=package://Robot/visualSTL/RR Wheel.STL
Joints:
- joint Chassis-FL Wheel: type Continuous -> continuous
- joint Chassis-FR Wheel: type Continuous -> continuous
- joint Chassis-RL Wheel: type Continuous -> continuous
- joint Chassis-RR Wheel: type Continuous -> continuous
